Commit message: Fix rename issues and change planning offset to 16.5 cm

File: ur10_gripper_description/urdf/ur10.urdf.xacro (robot description, xacro)
@@ -299,5 +299,5 @@
     <link name="${prefix}gripperOffset"/>
     <joint name="${prefix}ee_link2GripperOffset" type="fixed">
-      <origin xyz="0.18 0 0" rpy="0 0 0"/>
+      <origin xyz="0.165 0 0" rpy="0 0 0"/>
       <parent link="${prefix}ee_link"/>
       <child link="${prefix}gripperOffset"/>

File: ur10_gripper_description/urdf/ur10_gripper.urdf.xacro (robot description, xacro)
@@ -5,7 +5,7 @@
   <xacro:include filename="$(find ur_description)/urdf/common.gazebo.xacro" />
   <!-- ur10 -->
-  <xacro:include filename="$(find ur10_c2gripper)/urdf/ur10.urdf.xacro" />
+  <xacro:include filename="$(find ur10_gripper_description)/urdf/ur10.urdf.xacro" />
   <!-- gripper -->
-  <xacro:include filename="$(find ur10_c2gripper)/urdf/robotiq_c2_model.urdf" />
+  <xacro:include filename="$(find ur10_gripper_description)/urdf/robotiq_c2_model.urdf" />
   <!-- arm -->
 <xacro:ur10_robot prefix="" joint_limited="true" shoulder_pan_lower_limit="${-pi}" shoulder_pan_upper_limit="${pi}" shoulder_lift_lower_limit="${-pi}" shoulder_lift_upper_limit="${pi}" elbow_joint_lower_limit="${-pi}" elbow_joint_upper_limit="${pi}" wrist_1_lower_limit="${-pi}" wrist_1_upper_limit="${pi}" wrist_2_lower_limit="${-pi}" wrist_2_upper_limit="${pi}" wrist_3_lower_limit="${-pi}" wrist_3_upper_limit="${pi}"/>
