Commit message: Modified urdf and added static frame to flip the arm

File: ur10_gripper_description/urdf/robotiq_c2_model.urdf (robot description, URDF)
Before this commit: robot robotiq_c2_model, 10 links, 9 joints
Links:
- link robotiq_85_adapter_link: geometry collision mesh filename=package://robotiq_c2_model_visualization/meshes/robotiq_c2/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; visual mesh filename=package://robotiq_c2_model_visualization/meshes/robotiq_c2/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
- link robotiq_85_base_link: geometry collision mesh filename=package://robotiq_c2_model_visualization/meshes/robotiq_c2/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; visual mesh filename=package://robotiq_c2_model_visualization/meshes/robotiq_c2/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
- link robotiq_85_left_finger_link: geometry collision mesh filename=package://robotiq_c2_model_visualization/meshes/robotiq_c2/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; visual mesh filename=package://robotiq_c2_model_visualization/meshes/robotiq_c2/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
- link robotiq_85_left_finger_tip_link: geometry collision mesh filename=package://robotiq_c2_model_visualization/meshes/robotiq_c2/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; visual mesh filename=package://robotiq_c2_model_visualization/meshes/robotiq_c2/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
- link robotiq_85_left_inner_knuckle_link: geometry collision mesh filename=package://robotiq_c2_model_visualization/meshes/robotiq_c2/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; visual mesh filename=package://robotiq_c2_model_visualization/meshes/robotiq_c2/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
- link robotiq_85_left_knuckle_link: geometry collision mesh filename=package://robotiq_c2_model_visualization/meshes/robotiq_c2/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; visual mesh filename=package://robotiq_c2_model_visualization/meshes/robotiq_c2/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
- link robotiq_85_right_finger_link: geometry collision mesh filename=package://robotiq_c2_model_visualization/meshes/robotiq_c2/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; visual mesh filename=package://robotiq_c2_model_visualization/meshes/robotiq_c2/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
- link robotiq_85_right_finger_tip_link: geometry collision mesh filename=package://robotiq_c2_model_visualization/meshes/robotiq_c2/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; visual mesh filename=package://robotiq_c2_model_visualization/meshes/robotiq_c2/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
- link robotiq_85_right_inner_knuckle_link: geometry collision mesh filename=package://robotiq_c2_model_visualization/meshes/robotiq_c2/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; visual mesh filename=package://robotiq_c2_model_visualization/meshes/robotiq_c2/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
- link robotiq_85_right_knuckle_link: geometry collision mesh filename=package://robotiq_c2_model_visualization/meshes/robotiq_c2/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; visual mesh filename=package://robotiq_c2_model_visualization/meshes/robotiq_c2/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

File: ur10_gripper_description/urdf/ur10_gripper.urdf.xacro (robot description, xacro)
@@ -19,5 +19,5 @@
     <parent link="ee_link" />
     <child link = "robotiq_85_adapter_link" />
-    <origin xyz="0.0 0.0 0.0" rpy="0.0 0.0 0.0" />
+    <origin xyz="0.0 0.0 0.0" rpy="0.0 3.141592 0.0" />
   </joint>
 </robot>
