Commit message: #1 Deleted faiz ur_modern_driver folder.

File: ur10_gripper_description/urdf/ur10_gripper.urdf.xacro (robot description, xacro)
@@ -19,5 +19,5 @@
     <parent link="ee_link" />
     <child link = "robotiq_85_adapter_link" />
-    <origin xyz="0.0 0.0 0.0" rpy="0.0 3.141592 0.0" />
+    <origin xyz="0.0 0.0 0.0" rpy="0.0 0.0 0.0" />
   </joint>
 </robot>
